Commit message: Edit robot urdf xacro

File: gazebo_env/model/robot.xacro (robot description, xacro)
@@ -21,3 +21,14 @@
 <xacro:property name="wheel_mass" value="${wheel_density*pi*wheel_link_radius*wheel_link_radius*wheel_link_length}" />
 <!-- Moments of inertia of wheel -->
+<xacro:property name="Iz_wheel" value="${0.5*wheel_mass*wheel_link_radius*wheel_link_radius}" /> <!-- MI about cylindrical axis-->
+<xacro:property name="I_wheel"
+value = "${(1.0/12.0)*wheel_mass*(3.0*wheel_link_radius*wheel_link_radius + wheel_link_length*wheel_link_length)" />
+<!-- Inertia of wheel -->
+<xacro:property name="inertia_wheel">
+    <inertial>
+        <origin rpy="0 0 0" xyz="0 0 0" />
+        <mass value="${wheel_mass}"/>
+        <inertia ixx = "${I_wheel}" ixy = "0.0" ixz = "0.0" iyy = "${I_wheel}" iyz = "0" izz = "${Iz_wheel}" />
+    </inertial>
+</xacro:property>
 </robot>

Commit message: Edit robot urdf xacro

File: gazebo_env/model/robot.xacro (robot description, xacro)
@@ -16,5 +16,5 @@
 <xacro:property name="wheel_density" value="2700"/>
 <!-- Pi Constant -->
-<xacro:property name="pi" value="3.14159265"/>
+<xacro:property name="pi_const" value="3.14159265"/>
 <!-- Robot Body & wheel mass -->
 <xacro:property name="body_mass" value="${body_density*body_link_x_dim*body_link_y_dim*body_link_z_dim}" />
@@ -32,3 +32,37 @@
     </inertial>
 </xacro:property>
+<!-- Include extra Gazebo options & motion control driver  -->
+<xacro:include filename="$(find gazebo_env)/model/robot.gazebo" />
+<!-- ################################################# -->
+<!-- LINKS & JOINTS -->
+<!-- ################################################# -->
+<!-- Dummy link -->
+<link name="dummy" />
+<joint name= "dummy_joint" type="fixed">
+    <parent link="dummy" />
+    <child  link="body_link" />
+</joint>
+<!-- Body Link -->
+<link name="body_link" >
+    <visual>
+        <geometry>
+            <box size="$(body_link_x_dim) $(body_linky_dim) $(body_link_z_dim)" />
+        </geometry>
+    <origin rpy="0 0 0" xyz="0 0 0" />
+    </visual>
+    <collision>
+        <geometry>
+            <box size="$(body_link_x_dim) $(body_link_y_dim) $(body_link_z_dim)" />
+        </geometry>
+    </collision>
+    <inertial>
+        <origin rpy="0 0 0" xyz="0 0 0" />
+        <mass value="$(body_mass)" />
+        <inertia    ixx="${(1/12)*body_mass*(body_link_y_dim*body_link_y_dim + body_link_z_dim*body_link_z_dim)}"
+                    iyy="${(1/12)*body_mass*(body_link_x_dim*body_link_x_dim + body_link_z_dim*body_link_z_dim)}"
+                    izz="${(1/12)*body_mass*(body_link_y_dim*body_link_y_dim + body_link_x_dim*body_link_x_dim)}"
+                    ixy="0" ixz="0" iyz="0"
+        />
+    </inertial>
+</link>
 </robot>

Commit message: Final Edit urdf

File: gazebo_env/model/robot.xacro (robot description, xacro)
@@ -66,3 +66,107 @@
     </inertial>
 </link>
+<!-- Rear wheel Right (rwr)-->
+<!-- Joint -->
+<joint name="rwr_joint" type="continuous" >
+    <parent link="body_link" />
+    <child  link="rwr_link"  />
+    <origin xyz="${-body_link_x_dim/2} ${-(body_link_y_dim/2 + wheel_link_length/2)} ${wheel_link_z_loc}" rpy = "0 0 0" />
+    <axis xyz = "0 1 0"/> <!-- Revolves around y axis-->
+    <limit effort="1000" velocity="1000"/>
+    <dynamics damping="1.0" friction="1.0" />
+</joint>
+<!-- Link -->
+<link name="rwr_link">
+    <visual>
+        <origin rpy="${pi_const/2} 0 0" xyz="0 0 0" /> <!-- Rotate by 90deg -->
+        <geometry>
+            <cylinder length="${wheel_link_length}" radius="${wheel_link_radius}" />
+        </geometry>
+    </visual>
+    <collision>
+        <origin rpy="${pi_const/2} 0 0" xyz="0 0 0" />
+        <geometry>
+            <cylinder length="${wheel_link_length}" radius="${wheel_link_radius}" />
+        </geometry>
+    </collision>
+    <xacro:inertia_wheel />
+</link>
+<!-- Rear wheel left (rwl) -->
+<!-- Joint -->
+<joint name="rwl_joint" type="continuous" >
+    <parent link="body_link" />
+    <child  link="rwl_link"  />
+    <origin xyz="${-body_link_x_dim/2} ${(body_link_y_dim/2 + wheel_link_length/2)} ${wheel_link_z_loc}" rpy = "0 0 0" />
+    <axis xyz = "0 1 0"/> <!-- Revolves around y axis-->
+    <limit effort="1000" velocity="1000"/>
+    <dynamics damping="1.0" friction="1.0" />
+</joint>
+<!-- Link  -->
+<link name="rwl_link">
+    <visual>
+        <origin rpy="${pi_const/2} 0 0" xyz="0 0 0" /> <!-- Rotate by 90deg -->
+        <geometry>
+            <cylinder length="${wheel_link_length}" radius="${wheel_link_radius}" />
+        </geometry>
+    </visual>
+    <collision>
+        <origin rpy="${pi_const/2} 0 0" xyz="0 0 0" />
+        <geometry>
+            <cylinder length="${wheel_link_length}" radius="${wheel_link_radius}" />
+        </geometry>
+    </collision>
+    <xacro:inertia_wheel />
+</link>
+<!-- Front Wheel right (fwr) -->
+<!-- Joint -->
+<joint name="fwr_joint" type="continuous" >
+    <parent link="body_link" />
+    <child  link="fwr_link"  />
+    <origin xyz="${body_link_x_dim/2} ${-(body_link_y_dim/2 + wheel_link_length/2)} ${wheel_link_z_loc}" rpy = "0 0 0" />
+    <axis xyz = "0 1 0"/> <!-- Revolves around y axis-->
+    <limit effort="1000" velocity="1000"/>
+    <dynamics damping="1.0" friction="1.0" />
+</joint>
+<!-- Link  -->
+<link name="fwr_link">
+    <visual>
+        <origin rpy="${pi_const/2} 0 0" xyz="0 0 0" /> <!-- Rotate by 90deg -->
+        <geometry>
+            <cylinder length="${wheel_link_length}" radius="${wheel_link_radius}" />
+        </geometry>
+    </visual>
+    <collision>
+        <origin rpy="${pi_const/2} 0 0" xyz="0 0 0" />
+        <geometry>
+            <cylinder length="${wheel_link_length}" radius="${wheel_link_radius}" />
+        </geometry>
+    </collision>
+    <xacro:inertia_wheel />
+</link>
+<!-- Front Wheel left (fwl) -->
+<!-- Joint  -->
+<joint name="fwl_joint" type="continuous" >
+    <parent link="body_link" />
+    <child  link="fwl_link"  />
+    <origin xyz="${body_link_x_dim/2} ${(body_link_y_dim/2 + wheel_link_length/2)} ${wheel_link_z_loc}" rpy = "0 0 0" />
+    <axis xyz = "0 1 0"/> <!-- Revolves around y axis-->
+    <limit effort="1000" velocity="1000"/>
+    <dynamics damping="1.0" friction="1.0" />
+</joint>
+<!-- Link  -->
+<link name="fwl_link">
+    <visual>
+        <origin rpy="${pi_const/2} 0 0" xyz="0 0 0" /> <!-- Rotate by 90deg -->
+        <geometry>
+            <cylinder length="${wheel_link_length}" radius="${wheel_link_radius}" />
+        </geometry>
+    </visual>
+    <collision>
+        <origin rpy="${pi_const/2} 0 0" xyz="0 0 0" />
+        <geometry>
+            <cylinder length="${wheel_link_length}" radius="${wheel_link_radius}" />
+        </geometry>
+    </collision>
+    <xacro:inertia_wheel />
+</link>
 </robot>

Commit message: Add dependencies and install params in cmakelist, Corrections in xacro file, Add launch file

File: gazebo_env/model/robot.xacro (robot description, xacro)
@@ -47,5 +47,5 @@
     <visual>
         <geometry>
-            <box size="$(body_link_x_dim) $(body_linky_dim) $(body_link_z_dim)" />
+            <box size="${body_link_x_dim} ${body_linky_dim} ${body_link_z_dim}" />
         </geometry>
     <origin rpy="0 0 0" xyz="0 0 0" />
@@ -53,5 +53,5 @@
     <collision>
         <geometry>
-            <box size="$(body_link_x_dim) $(body_link_y_dim) $(body_link_z_dim)" />
+            <box size="${body_link_x_dim} ${body_link_y_dim} ${body_link_z_dim}" />
         </geometry>
     </collision>

Commit message: xacro file corrections

File: gazebo_env/model/robot.xacro (robot description, xacro)
@@ -23,7 +23,7 @@
 <xacro:property name="Iz_wheel" value="${0.5*wheel_mass*wheel_link_radius*wheel_link_radius}" /> <!-- MI about cylindrical axis-->
 <xacro:property name="I_wheel"
-value = "${(1.0/12.0)*wheel_mass*(3.0*wheel_link_radius*wheel_link_radius + wheel_link_length*wheel_link_length)" />
+value = "${(1.0/12.0)*wheel_mass*(3.0*wheel_link_radius*wheel_link_radius + wheel_link_length*wheel_link_length)}" />
 <!-- Inertia of wheel -->
-<xacro:property name="inertia_wheel">
+<xacro:macro name="inertia_wheel">
     <inertial>
         <origin rpy="0 0 0" xyz="0 0 0" />
@@ -31,5 +31,5 @@
         <inertia ixx = "${I_wheel}" ixy = "0.0" ixz = "0.0" iyy = "${I_wheel}" iyz = "0" izz = "${Iz_wheel}" />
     </inertial>
-</xacro:property>
+</xacro:macro>
 <!-- Include extra Gazebo options & motion control driver  -->
 <xacro:include filename="$(find gazebo_env)/model/robot.gazebo" />
@@ -47,5 +47,5 @@
     <visual>
         <geometry>
-            <box size="${body_link_x_dim} ${body_linky_dim} ${body_link_z_dim}" />
+            <box size="${body_link_x_dim} ${body_link_y_dim} ${body_link_z_dim}" />
         </geometry>
     <origin rpy="0 0 0" xyz="0 0 0" />
@@ -58,5 +58,5 @@
     <inertial>
         <origin rpy="0 0 0" xyz="0 0 0" />
-        <mass value="$(body_mass)" />
+        <mass value="${body_mass}" />
         <inertia    ixx="${(1/12)*body_mass*(body_link_y_dim*body_link_y_dim + body_link_z_dim*body_link_z_dim)}"
                     iyy="${(1/12)*body_mass*(body_link_x_dim*body_link_x_dim + body_link_z_dim*body_link_z_dim)}"

Commit message: Minor Updates

File: gazebo_env/model/robot.xacro (robot description, xacro)
@@ -4,4 +4,5 @@
 <!-- Chetan VJ© -->
 <robot name = "differential_drive_robot" xmlns:xacro = "http://www.ros.org/wiki/xacro">
+<xacro:property name="camera_name" value="cam1"/>
 <!-- Body Dimensions (units in meters)-->
 <xacro:property name="body_link_x_dim" value="0.79"/>
@@ -171,3 +172,23 @@
     <xacro:inertia_wheel />
 </link>
+<!-- Camera Link -->
+<joint name = "camera_joint" type="fixed">
+    <parent link="body_link"/>
+    <child link="camera_link" />
+    <origin xyz="${body_link_x_dim/2} 0 ${body_link_z_dim/2}" />
+</joint>
+<link name="camera_link">
+    <visual>
+        <geometry>
+            <box size="0.010 0.03 0.03"/>
+        </geometry>
+        <material name="red"/>
+    </visual>
+</link>
+<joint name="camera_optical_joint" type="fixed">
+        <parent link="camera_link"/>
+        <child link="camera_link_optical"/>
+        <origin xyz="0 0 0" rpy="${-pi/2} 0 ${-pi/2}"/>
+</joint>
+<link name="camera_link_optical"></link>
 </robot>

Commit message: update camera co'ods

File: gazebo_env/model/robot.xacro (robot description, xacro)
@@ -176,5 +176,5 @@
     <parent link="body_link"/>
     <child link="camera_link" />
-    <origin xyz="${body_link_x_dim/2} 0 ${body_link_z_dim/2}" />
+    <origin xyz="${body_link_x_dim/2} 0 ${body_link_z_dim/2}" rpy="0 0 0"/>
 </joint>
 <link name="camera_link">

Commit message: Camera topic fix

File: gazebo_env/model/robot.xacro (robot description, xacro)
@@ -183,5 +183,5 @@
             <box size="0.010 0.03 0.03"/>
         </geometry>
-        <material name="red"/>
+        <!-- <material name="red"/> -->
     </visual>
 </link>

Commit message: Add Improvements

File: gazebo_env/model/robot.xacro (robot description, xacro)
@@ -12,4 +12,5 @@
 <xacro:property name="wheel_link_radius" value="0.125"/>
 <xacro:property name="wheel_link_length" value="0.05"/>
+<xacro:property name="wheel_mesh_scale"  value="${wheel_link_radius/125}" />
 <xacro:property name="wheel_link_z_loc" value="-0.05"/>
 <!-- Material Density -->
@@ -81,7 +82,7 @@
 <link name="rwr_link">
     <visual>
-        <origin rpy="${pi_const/2} 0 0" xyz="0 0 0" /> <!-- Rotate by 90deg -->
+        <origin rpy="${pi_const/2} 0 ${-pi_const/2}" xyz="0 0 0" /> <!-- Rotate by 90deg -->
         <geometry>
-            <cylinder length="${wheel_link_length}" radius="${wheel_link_radius}" />
+            <mesh filename="file://$(find gazebo_env)/meshes/wheel.stl" scale="${wheel_mesh_scale} ${wheel_mesh_scale} ${wheel_mesh_scale}" />
         </geometry>
     </visual>
@@ -107,7 +108,7 @@
 <link name="rwl_link">
     <visual>
-        <origin rpy="${pi_const/2} 0 0" xyz="0 0 0" /> <!-- Rotate by 90deg -->
+        <origin rpy="${pi_const/2} 0 ${pi_const/2}" xyz="0 0 0" /> <!-- Rotate by 90deg -->
         <geometry>
-            <cylinder length="${wheel_link_length}" radius="${wheel_link_radius}" />
+            <mesh filename="file://$(find gazebo_env)/meshes/wheel.stl" scale="${wheel_mesh_scale} ${wheel_mesh_scale} ${wheel_mesh_scale}" />
         </geometry>
     </visual>
@@ -133,7 +134,7 @@
 <link name="fwr_link">
     <visual>
-        <origin rpy="${pi_const/2} 0 0" xyz="0 0 0" /> <!-- Rotate by 90deg -->
+        <origin rpy="${pi_const/2} 0 ${-pi_const/2}" xyz="0 0 0" /> <!-- Rotate by 90deg -->
         <geometry>
-            <cylinder length="${wheel_link_length}" radius="${wheel_link_radius}" />
+            <mesh filename="file://$(find gazebo_env)/meshes/wheel.stl" scale="${wheel_mesh_scale} ${wheel_mesh_scale} ${wheel_mesh_scale}" />
         </geometry>
     </visual>
@@ -159,7 +160,7 @@
 <link name="fwl_link">
     <visual>
-        <origin rpy="${pi_const/2} 0 0" xyz="0 0 0" /> <!-- Rotate by 90deg -->
+        <origin rpy="${pi_const/2} 0 ${pi_const/2}" xyz="0 0 0" /> <!-- Rotate by 90deg -->
         <geometry>
-            <cylinder length="${wheel_link_length}" radius="${wheel_link_radius}" />
+            <mesh filename="file://$(find gazebo_env)/meshes/wheel.stl" scale="${wheel_mesh_scale} ${wheel_mesh_scale} ${wheel_mesh_scale}" />
         </geometry>
     </visual>
@@ -176,5 +177,5 @@
     <parent link="body_link"/>
     <child link="camera_link" />
-    <origin xyz="${body_link_x_dim/2} 0 ${body_link_z_dim/2}" rpy="0 0 0"/>
+    <origin xyz="${body_link_x_dim/2} 0 ${body_link_z_dim/2}" />
 </joint>
 <link name="camera_link">

Commit message: Minor improvements in Bot description

File: gazebo_env/model/robot.xacro (robot description, xacro)
@@ -11,5 +11,5 @@
 <!-- Wheel Dimensions -->
 <xacro:property name="wheel_link_radius" value="0.125"/>
-<xacro:property name="wheel_link_length" value="0.05"/>
+<xacro:property name="wheel_link_length" value="1"/>
 <xacro:property name="wheel_mesh_scale"  value="${wheel_link_radius/125}" />
 <xacro:property name="wheel_link_z_loc" value="-0.05"/>
@@ -82,5 +82,5 @@
 <link name="rwr_link">
     <visual>
-        <origin rpy="${pi_const/2} 0 ${-pi_const/2}" xyz="0 0 0" /> <!-- Rotate by 90deg -->
+        <origin rpy="${pi_const/2} 0 ${-pi_const/2}" xyz="0 0.5 0" /> <!-- Rotate by 90deg -->
         <geometry>
             <mesh filename="file://$(find gazebo_env)/meshes/wheel.stl" scale="${wheel_mesh_scale} ${wheel_mesh_scale} ${wheel_mesh_scale}" />
@@ -108,5 +108,5 @@
 <link name="rwl_link">
     <visual>
-        <origin rpy="${pi_const/2} 0 ${pi_const/2}" xyz="0 0 0" /> <!-- Rotate by 90deg -->
+        <origin rpy="${pi_const/2} 0 ${pi_const/2}" xyz="0 -0.5 0" /> <!-- Rotate by 90deg -->
         <geometry>
             <mesh filename="file://$(find gazebo_env)/meshes/wheel.stl" scale="${wheel_mesh_scale} ${wheel_mesh_scale} ${wheel_mesh_scale}" />
@@ -134,5 +134,5 @@
 <link name="fwr_link">
     <visual>
-        <origin rpy="${pi_const/2} 0 ${-pi_const/2}" xyz="0 0 0" /> <!-- Rotate by 90deg -->
+        <origin rpy="${pi_const/2} 0 ${-pi_const/2}" xyz="0 0.5 0" /> <!-- Rotate by 90deg -->
         <geometry>
             <mesh filename="file://$(find gazebo_env)/meshes/wheel.stl" scale="${wheel_mesh_scale} ${wheel_mesh_scale} ${wheel_mesh_scale}" />
@@ -160,5 +160,5 @@
 <link name="fwl_link">
     <visual>
-        <origin rpy="${pi_const/2} 0 ${pi_const/2}" xyz="0 0 0" /> <!-- Rotate by 90deg -->
+        <origin rpy="${pi_const/2} 0 ${pi_const/2}" xyz="0 -0.5 0" /> <!-- Rotate by 90deg --> <!-- xyz values purely for visualization, doesn't affect simulation -->
         <geometry>
             <mesh filename="file://$(find gazebo_env)/meshes/wheel.stl" scale="${wheel_mesh_scale} ${wheel_mesh_scale} ${wheel_mesh_scale}" />

Commit message: Add Lidar Sensor to Bot

File: gazebo_env/model/robot.xacro (robot description, xacro)
@@ -193,3 +193,21 @@
 </joint>
 <link name="camera_link_optical"></link>
+<!-- Lidar Link  -->
+<joint name="lidar_joint" type="fixed">
+    <parent link="body_link" />
+    <child link="lidar_link" />
+    <origin xyz="${-body_link_x_dim/2+0.1} 0 ${body_link_z_dim/2+0.02}" />
+</joint>
+<link name="lidar_link">
+    <visual>
+        <geometry>
+            <cylinder radius="0.08" length="0.04"/>
+        </geometry>
+    </visual>
+    <collision>
+        <geometry>
+            <cylinder radius="0.08" length="0.04"/>
+        </geometry>
+    </collision>
+</link>
 </robot>

Commit message: Add SLAM functionality using slam_toolbox

File: gazebo_env/model/robot.xacro (robot description, xacro)
@@ -42,4 +42,12 @@
 <!-- Dummy link -->
 <link name="dummy" />
+<!-- The base_footprint link is required by the slam toolbox, as mentioned  -->
+<!-- in the mapper_params_ yaml file -->
+<joint name="base_footprint_joint" type="fixed">
+    <parent link="dummy"/>
+    <child link="base_footprint"/>
+    <origin xyz="0 0 0" rpy="0 0 0"/>
+</joint>
+<link name="base_footprint" />
 <joint name= "dummy_joint" type="fixed">
     <parent link="dummy" />

Commit message: Add new mesh for body

File: gazebo_env/model/robot.xacro (robot description, xacro)
@@ -58,5 +58,5 @@
     <visual>
         <geometry>
-            <box size="${body_link_x_dim} ${body_link_y_dim} ${body_link_z_dim}" />
+            <mesh filename="file://$(find gazebo_env)/meshes/body.stl" scale="${wheel_mesh_scale} ${wheel_mesh_scale} ${wheel_mesh_scale}" />
         </geometry>
     <origin rpy="0 0 0" xyz="0 0 0" />
@@ -82,5 +82,5 @@
     <parent link="body_link" />
     <child  link="rwr_link"  />
-    <origin xyz="${-body_link_x_dim/2} ${-(body_link_y_dim/2 + wheel_link_length/2)} ${wheel_link_z_loc}" rpy = "0 0 0" />
+    <origin xyz="${-body_link_x_dim/2+0.1} ${-(body_link_y_dim/2 + wheel_link_length/2)} ${wheel_link_z_loc+0.05}" rpy = "0 0 0" />
     <axis xyz = "0 1 0"/> <!-- Revolves around y axis-->
     <limit effort="1000" velocity="1000"/>
@@ -108,5 +108,5 @@
     <parent link="body_link" />
     <child  link="rwl_link"  />
-    <origin xyz="${-body_link_x_dim/2} ${(body_link_y_dim/2 + wheel_link_length/2)} ${wheel_link_z_loc}" rpy = "0 0 0" />
+    <origin xyz="${-body_link_x_dim/2+0.1} ${(body_link_y_dim/2 + wheel_link_length/2)} ${wheel_link_z_loc+0.05}" rpy = "0 0 0" />
     <axis xyz = "0 1 0"/> <!-- Revolves around y axis-->
     <limit effort="1000" velocity="1000"/>
@@ -134,5 +134,5 @@
     <parent link="body_link" />
     <child  link="fwr_link"  />
-    <origin xyz="${body_link_x_dim/2} ${-(body_link_y_dim/2 + wheel_link_length/2)} ${wheel_link_z_loc}" rpy = "0 0 0" />
+    <origin xyz="${body_link_x_dim/2-0.1} ${-(body_link_y_dim/2 + wheel_link_length/2)} ${wheel_link_z_loc+0.05}" rpy = "0 0 0" />
     <axis xyz = "0 1 0"/> <!-- Revolves around y axis-->
     <limit effort="1000" velocity="1000"/>
@@ -160,5 +160,5 @@
     <parent link="body_link" />
     <child  link="fwl_link"  />
-    <origin xyz="${body_link_x_dim/2} ${(body_link_y_dim/2 + wheel_link_length/2)} ${wheel_link_z_loc}" rpy = "0 0 0" />
+    <origin xyz="${body_link_x_dim/2-0.1} ${(body_link_y_dim/2 + wheel_link_length/2)} ${wheel_link_z_loc+0.05}" rpy = "0 0 0" />
     <axis xyz = "0 1 0"/> <!-- Revolves around y axis-->
     <limit effort="1000" velocity="1000"/>
@@ -205,5 +205,5 @@
     <parent link="body_link" />
     <child link="lidar_link" />
-    <origin xyz="${-body_link_x_dim/2+0.1} 0 ${body_link_z_dim/2+0.02}" />
+    <origin xyz="${-body_link_x_dim/2+0.1} 0 ${body_link_z_dim/2+0.09}" />
 </joint>
 <link name="lidar_link">

Commit message: Update README & minor changes to xacro

File: gazebo_env/model/robot.xacro (robot description, xacro)
@@ -189,7 +189,7 @@
 <link name="camera_link">
     <visual>
-        <geometry>
+        <!-- <geometry>
             <box size="0.010 0.03 0.03"/>
-        </geometry>
+        </geometry> -->
         <!-- <material name="red"/> -->
     </visual>
